Commit message: publish official release

File: assets/panda/franka_robotiq2f85.urdf (robot description, URDF)
Before this commit: robot panda, 17 links, 16 joints
Joints:
- joint finger_joint: limit (none) -> lower=0 upper=0.725 effort=1000 velocity=2.0
- joint left_inner_finger_joint: limit (none) -> lower=-0.8757 upper=0 effort=1000 velocity=2.0
- joint left_inner_knuckle_joint: limit (none) -> lower=0 upper=0.8757 effort=1000 velocity=2.0
- joint panda_joint1: limit (none) -> lower=-2.8973 upper=2.8973 effort=87 velocity=2.1750
- joint panda_joint2: limit (none) -> lower=-1.7628 upper=1.7628 effort=87 velocity=2.1750
- joint panda_joint3: limit (none) -> lower=-2.8973 upper=2.8973 effort=87 velocity=2.1750
- joint panda_joint4: limit (none) -> lower=-3.0718 upper=-0.0698 effort=87 velocity=2.1750
- joint panda_joint5: limit (none) -> lower=-2.8973 upper=2.8973 effort=12 velocity=2.6100
- joint panda_joint6: limit (none) -> lower=-0.0175 upper=3.7525 effort=12 velocity=2.6100
- joint panda_joint7: limit (none) -> lower=-2.8973 upper=2.8973 effort=12 velocity=2.6100
- joint right_inner_finger_joint: limit (none) -> lower=0 upper=0.8757 effort=1000 velocity=2.0
- joint right_inner_knuckle_joint: limit (none) -> lower=-0.8757 upper=0 effort=1000 velocity=2.0
- joint right_outer_knuckle_joint: limit (none) -> lower=-0.8757 upper=0 effort=1000 velocity=2.0
